Commit message: Created cor URDF

File: description/robot_core.xacro (robot description, xacro)
@@ -1,4 +1,5 @@
 <?xml version="1.0"?>
 <robot xmlns:xacro="http://www.ros.org/wiki/xacro" >
+    <xacro:include filename='inertial_macros.xacro'/>
     <!-- COLOR -->
     <material name="white">
@@ -16,5 +17,5 @@
     <link name="base_link">
     </link>
-    <!-- CHASSIS LINK-->
+    <!-- CHASSIS -->
     <joint name="chassis_joint" type="fixed">
         <parent link="base_link"/>
@@ -30,4 +31,14 @@
             <material name="white"/>
         </visual>
+        <collision>
+            <origin xyz="0 0 0.15"/>
+            <geometry>
+                <cylinder radius="0.24" length="0.3"/>
+            </geometry>
+            <material name="white"/>
+        </collision>
+        <xacro:inertial_cylinder mass="0.5" radius="0.24" length="0.3">
+            <origin xyz="0 0 0.15" rpy="0 0 0"/>
+        </xacro:inertial_cylinder>
     </link>
     <!-- LEFT WHEEL -->
@@ -41,8 +52,17 @@
         <visual>
             <geometry>
-                <cylinder length="0.05" radius="0.09" />
+                <cylinder length="0.05" radius="0.05" />
             </geometry>
             <material name="blue"/>
         </visual>
+        <collision>
+            <geometry>
+                <cylinder length="0.05" radius="0.05" />
+            </geometry>
+            <material name="blue"/>
+        </collision>
+        <xacro:inertial_cylinder mass="1" length="0.05" radius="0.05">
+            <origin xyz="0 0 0" rpy="0 0 0"/>
+        </xacro:inertial_cylinder>
     </link>
     <!-- RIGHT WHEEL -->
@@ -56,16 +76,25 @@
         <visual>
             <geometry>
-                <cylinder length="0.05" radius="0.09" />
+                <cylinder length="0.05" radius="0.05" />
             </geometry>
             <material name="blue"/>
         </visual>
+        <collision>
+            <geometry>
+                <cylinder length="0.05" radius="0.05" />
+            </geometry>
+            <material name="blue"/>
+        </collision>
+        <xacro:inertial_cylinder mass="1" length="0.05" radius="0.05">
+            <origin xyz="0 0 0" rpy="0 0 0"/>
+        </xacro:inertial_cylinder>
     </link>
     <!-- CASTER WHEEL 1 -->
-    <joint name="caster_wheel_joint" type="fixed">
+    <joint name="caster_wheel_1_joint" type="fixed">
         <parent link="chassis"/>
-        <child link="caster_wheel"/>
-        <origin xyz="0.20 0 0" rpy="0 0 0"/>
+        <child link="caster_wheel_1"/>
+        <origin xyz="0.18 0 0" />
     </joint>
-    <link name="caster_wheel">
+    <link name="caster_wheel_1">
         <visual>
             <geometry>
@@ -74,4 +103,36 @@
             <material name="black"/>
         </visual>
+        <collision>
+            <geometry>
+                <sphere radius="0.05" />
+            </geometry>
+            <material name="black"/>
+        </collision>
+        <xacro:inertial_sphere mass="0.1" radius="0.05">
+            <origin xyz="0 0 0" rpy="0 0 0"/>
+        </xacro:inertial_sphere>
+    </link>
+    <!-- CASTER WHEEL 2 -->
+    <joint name="caster_wheel_2_joint" type="fixed">
+        <parent link="chassis"/>
+        <child link="caster_wheel_2"/>
+        <origin xyz="-0.18 0 0" />
+    </joint>
+    <link name="caster_wheel_2">
+        <visual>
+            <geometry>
+                <sphere radius="0.05" />
+            </geometry>
+            <material name="black"/>
+        </visual>
+        <collision>
+            <geometry>
+                <sphere radius="0.05" />
+            </geometry>
+            <material name="black"/>
+        </collision>
+        <xacro:inertial_sphere mass="0.1" radius="0.05">
+            <origin xyz="0 0 0" rpy="0 0 0"/>
+        </xacro:inertial_sphere>
     </link>
 </robot>

Commit message: Simulated Gazebo

File: description/robot_core.xacro (robot description, xacro)
@@ -42,4 +42,7 @@
         </xacro:inertial_cylinder>
     </link>
+    <gazebo reference="chassis">
+        <material>Gazebo/White</material>
+    </gazebo>
     <!-- LEFT WHEEL -->
     <joint name="left_wheel_joint" type="continuous">
@@ -66,4 +69,7 @@
         </xacro:inertial_cylinder>
     </link>
+    <gazebo reference="left_wheel">
+        <material>Gazebo/Blue</material>
+    </gazebo>
     <!-- RIGHT WHEEL -->
     <joint name="right_wheel_joint" type="continuous">
@@ -90,4 +96,7 @@
         </xacro:inertial_cylinder>
     </link>
+    <gazebo reference="right_wheel">
+        <material>Gazebo/Blue</material>
+    </gazebo>
     <!-- CASTER WHEEL 1 -->
     <joint name="caster_wheel_1_joint" type="fixed">
@@ -113,4 +122,9 @@
         </xacro:inertial_sphere>
     </link>
+    <gazebo reference="caster_wheel_1">
+        <material>Gazebo/Black</material>
+        <mu1 value="0.001"/>
+        <mu2 value="0.001"/>
+    </gazebo>
     <!-- CASTER WHEEL 2 -->
     <joint name="caster_wheel_2_joint" type="fixed">
@@ -136,3 +150,8 @@
         </xacro:inertial_sphere>
     </link>
+    <gazebo reference="caster_wheel_2">
+        <material>Gazebo/Black</material>
+        <mu1 value="0.001"/>
+<mu2 value="0.001"/>
+    </gazebo>
 </robot>
